Commit message: updated rov model, depth sensor, controller

File: nemesys_surveillance/urdf/nemesys.urdf.xacro (robot description, xacro)
@@ -25,36 +25,32 @@
     </material>
     <!-- base_link DEFINITION -->
-    <link name="base_link" />
-    <!-- main_body_link_nemesys DEFINITION -->
-    <link name="main_body_link_nemesys">
-        <visual>
-            <geometry>
-                <mesh filename="package://nemesys_surveillance/meshes/main_body_link_nemesys.STL"
-                      scale="${scale_size} ${scale_size} ${scale_size}" />
-            </geometry>
-            <origin xyz="0 0 0" rpy="${pi/2} 0 0" />
+    <!-- <link name="base_link" /> -->
+    <!-- base_link DEFINITION -->
+    <link name="base_link">
+        <visual>
+            <geometry>
+                <mesh filename="package://nemesys_surveillance/meshes/NemeSys_adjusted.stl"
+                      scale="${scale_size} ${scale_size} ${scale_size}" />
+            </geometry>
+            <origin xyz="0 0 0" rpy="0 0 0" />
             <material name="Custom_Color" />
         </visual>
         <collision>
             <geometry>
-                <mesh filename="package://nemesys_surveillance/meshes/main_body_link_nemesys.STL"
-                      scale="${scale_size} ${scale_size} ${scale_size}" />
-            </geometry>
-            <origin xyz="0 0 0" rpy="${pi/2} 0 0" />
-        </collision>
-        <inertial>
-            <origin xyz="${scale_size*-0.8e-3} 0 ${scale_size*-4.55e-3}" rpy="0 0 0" />
-            <mass value="8.6" />
-            <inertia ixx="41763721.74e-9" ixy="76.64e-9" ixz="-1071029.52e-9"
-                     iyy="99391057.27e-9" iyz="603.74e-9"
-                     izz="101413261.83e-9" />
-        </inertial>
-    </link>
-    <!-- base_link TO main_body_link_nemesys JOINT DEFINITION -->
-    <joint name="base_to_main_body_joint" type="fixed">
-        <parent link="base_link" />
-        <child link="main_body_link_nemesys" />
-        <origin xyz="0 0 ${scale_size*tube_od/2}" rpy="0 0 0" />
-    </joint>
+                <mesh filename="package://nemesys_surveillance/meshes/NemeSys_adjusted.stl"
+                      scale="${scale_size} ${scale_size} ${scale_size}" />
+            </geometry>
+            <origin xyz="0 0 0" rpy="0 0 0" />
+        </collision>
+        <inertial>
+            <!-- Put COM at 0 initially unless you KNOW it's offset -->
+            <origin xyz="0 0 0" rpy="0 0 0"/>
+            <mass value="8.6"/>
+            <inertia
+                ixx="0.02930236" ixy="0.0" ixz="0.0"
+                iyy="0.07848640" iyz="0.0"
+                izz="0.07848640"/>
+        </inertial>
+    </link>
     <!-- front_right_thruster_link_nemesys DEFINITION -->
     <link name="front_right_thruster_link_nemesys">
@@ -82,9 +78,9 @@
         </inertial>
     </link>
-    <!-- main_body_link_nemesys TO front_right_thruster_link_nemesys JOINT DEFINITION -->
+    <!-- base_link TO front_right_thruster_link_nemesys JOINT DEFINITION -->
     <joint name="body_to_fr_thruster_joint" type="continuous">
-        <parent link="main_body_link_nemesys" />
+        <parent link="base_link" />
         <child link="front_right_thruster_link_nemesys" />
-        <origin xyz="${scale_size*-0.325} ${scale_size*0.24} 0" rpy="0 0 0"/>
+        <origin xyz="${scale_size*0.0} ${scale_size*-0.24} ${scale_size*0.0}" rpy="0 0 0"/>
         <axis xyz="0 0 1" />
     </joint>
@@ -114,9 +110,9 @@
         </inertial>
     </link>
-    <!-- main_body_link_nemesys TO front_left_thruster_link_nemesys JOINT DEFINITION -->
+    <!-- base_link TO front_left_thruster_link_nemesys JOINT DEFINITION -->
     <joint name="body_to_fl_thruster_joint" type="continuous">
-        <parent link="main_body_link_nemesys" />
+        <parent link="base_link" />
         <child link="front_left_thruster_link_nemesys" />
-        <origin xyz="${scale_size*-0.325} ${scale_size*-0.24} 0" rpy="0 0 0"/>
+        <origin xyz="${scale_size*0.0} ${scale_size*0.24} ${scale_size*0.0}" rpy="0 0 0"/>
         <axis xyz="0 0 1" />
     </joint>
@@ -146,9 +142,9 @@
         </inertial>
     </link>
-    <!-- main_body_link_nemesys TO rear_right_thruster_link_nemesys JOINT DEFINITION -->
+    <!-- base_link TO rear_right_thruster_link_nemesys JOINT DEFINITION -->
     <joint name="body_to_rr_thruster_joint" type="continuous">
-        <parent link="main_body_link_nemesys" />
+        <parent link="base_link" />
         <child link="rear_right_thruster_link_nemesys" />
-        <origin xyz="${scale_size*-0.61} ${scale_size*0.11} ${scale_size*0.004}" rpy="0 0 0"/>
+        <origin xyz="${scale_size*-0.25} ${scale_size*-0.11} ${scale_size*0.0}" rpy="0 0 0"/>
         <axis xyz="1 0 0" />
     </joint>
@@ -178,9 +174,9 @@
         </inertial>
     </link>
-    <!-- main_body_link_nemesys TO rear_left_thruster_link_nemesys JOINT DEFINITION -->
+    <!-- base_link TO rear_left_thruster_link_nemesys JOINT DEFINITION -->
     <joint name="body_to_rl_thruster_joint" type="continuous">
-        <parent link="main_body_link_nemesys" />
+        <parent link="base_link" />
         <child link="rear_left_thruster_link_nemesys" />
-        <origin xyz="${scale_size*-0.60058} ${scale_size*-0.11} ${scale_size*0.004}" rpy="0 0 0"/>
+        <origin xyz="${scale_size*-0.25} ${scale_size*0.11} ${scale_size*-0.0}" rpy="0 0 0"/>
         <axis xyz="1 0 0" />
     </joint>
@@ -208,9 +204,9 @@
         </inertial>
     </link>
-    <!-- main_body_link_nemesys TO downward_camera_link JOINT DEFINITION -->
+    <!-- base_link TO downward_camera_link JOINT DEFINITION -->
     <joint name="body_to_down_cam_joint" type="fixed">
-        <parent link="main_body_link_nemesys" />
+        <parent link="base_link" />
         <child link="downward_camera_link" />
-        <origin xyz="${scale_size*-0.04591} 0 ${scale_size*0.0687}" rpy="${-pi/2} ${-pi/2} 0"/>
+        <origin xyz="${scale_size*0.14591} 0 ${scale_size*-0.2687}" rpy="0 ${pi/2} 0"/>
     </joint>
     <!-- front_camera_link DEFINITION -->
@@ -237,9 +233,9 @@
         </inertial>
     </link>
-    <!-- main_body_link_nemesys TO front_camera_link JOINT DEFINITION -->
+    <!-- base_link TO front_camera_link JOINT DEFINITION -->
     <joint name="body_to_front_cam_joint" type="fixed">
-        <parent link="main_body_link_nemesys" />
+        <parent link="base_link" />
         <child link="front_camera_link" />
-        <origin xyz="${scale_size*0.186} 0 0" rpy="${pi} 0 0"/>
+        <origin xyz="${scale_size*0.32} 0 0" rpy="0 0 0"/>
     </joint>
     <!-- bar30_sensor_link DEFINITION -->
@@ -252,10 +248,10 @@
             <material name="Black" />
         </visual>
-        <collision>
-            <geometry>
-                <sphere radius = "${scale_size*0.001}"/>
-            </geometry>
-            <origin xyz="0 0 0" rpy="0 0 0" />
-        </collision>
+        <!-- <collision>
+            <geometry>
+                <sphere radius = "${scale_size*0.001}"/>
+            </geometry>
+            <origin xyz="0 0 0" rpy="0 0 0" />
+        </collision> -->
         <inertial>
             <origin xyz="0 0 0" rpy="0 0 0" />
@@ -266,9 +262,9 @@
         </inertial>
     </link>
-    <!-- main_body_link_nemesys TO bar30_sensor_link JOINT DEFINITION -->
+    <!-- base_link TO bar30_sensor_link JOINT DEFINITION -->
     <joint name="body_to_bar30_joint" type="fixed">
-        <parent link="main_body_link_nemesys" />
+        <parent link="base_link" />
         <child link="bar30_sensor_link" />
-        <origin xyz="${scale_size*-0.16684} 0 0" rpy="0 0 0"/>
+        <origin xyz="${scale_size*0} 0 ${scale_size*0.01}" rpy="0 0 0"/>
     </joint>
     <!-- imu_link DEFINITION -->
@@ -295,7 +291,7 @@
         </inertial>
     </link>
-    <!-- main_body_link_nemesys TO imu_link JOINT DEFINITION -->
+    <!-- base_link TO imu_link JOINT DEFINITION -->
     <joint name="body_to_imu_joint" type="fixed">
-        <parent link="main_body_link_nemesys" />
+        <parent link="base_link" />
         <child link="imu_link" />
         <origin xyz="0 0 0" rpy="0 0 0"/>
@@ -306,5 +302,5 @@
             <origin xyz="0 0 0" rpy="0 0 0"/>
             <geometry>
-            <cylinder radius="0.02" length="0.05"/>
+            <cylinder radius="0.01" length="0.03"/>
             </geometry>
             <material name="Green">
@@ -315,5 +311,5 @@
             <origin xyz="0 0 0" rpy="0 0 0"/>
             <geometry>
-            <cylinder radius="0.02" length="0.05"/>
+            <cylinder radius="0.01" length="0.03"/>
             </geometry>
         </collision>
@@ -329,5 +325,5 @@
     </link>
         <joint name="body_to_hydrophone_joint" type="fixed">
-        <parent link="main_body_link_nemesys"/>
+        <parent link="base_link"/>
         <child link="hydrophone_link"/>
         <origin xyz="0.0 0.0 0.0" rpy="0 0 0"/>
@@ -385,5 +381,5 @@
         </plugin>
     </gazebo>
-    <gazebo reference="main_body_link_nemesys">
+    <gazebo reference="base_link">
         <material>Gazebo/White</material>
     </gazebo>
@@ -552,26 +548,22 @@
     <!-- BAR30 SENSOR (DEPTH) PLUGIN -->
     <gazebo reference="bar30_sensor_link">
-    <sensor type="ray" name="depth_sensor">
-        <pose>0 0 0 0 0 0</pose>
-        <visualize>true</visualize>
-        <update_rate>10</update_rate>
-        <ray>
+        <sensor type="ray" name="depth_sensor">
+            <!-- Rotate so +X points to +Z (up) -->
+            <pose>0 0 0 0 -1.570796 0</pose>
+            <visualize>true</visualize>
+            <update_rate>10</update_rate>
+            <ray>
             <scan>
                 <horizontal>
-                    <samples>1</samples>
+                    <samples>61</samples>
                     <resolution>1</resolution>
-                    <min_angle>.000001</min_angle>
-                    <max_angle>0</max_angle>
+                    <min_angle>-0.261799</min_angle>  <!-- -15 deg -->
+                    <max_angle> 0.261799</max_angle>  <!-- +15 deg -->
                 </horizontal>
-                <vertical>
-                    <samples>2</samples>
-                    <resolution>1</resolution>
-                    <min_angle>-1.570796</min_angle>
-                    <max_angle>-1.570795</max_angle>
-                </vertical>
             </scan>
             <range>
-                <min>-100</min>
-                <max>100.0</max>
+                <!-- MUST be non-negative -->
+                <min>0.05</min>
+                <max>200.0</max>
                 <resolution>0.01</resolution>
             </range>
@@ -581,10 +573,10 @@
                 <stddev>0.01</stddev>
             </noise>
-        </ray>
-        <plugin name="gazebo_ros_head_hokuyo_controller" filename="libgazebo_ros_laser.so">
+            </ray>
+            <plugin name="gazebo_ros_laser" filename="libgazebo_ros_laser.so">
             <topicName>/raw_depth_data</topicName>
             <frameName>bar30_sensor_link</frameName>
-        </plugin>
-    </sensor>
+            </plugin>
+        </sensor>
     </gazebo>
     <!-- IMU PLUGIN -->

Commit message: status pub rewritten; COB & depth control revised

File: nemesys_surveillance/urdf/nemesys.urdf.xacro (robot description, xacro)
@@ -146,5 +146,5 @@
         <parent link="base_link" />
         <child link="rear_right_thruster_link_nemesys" />
-        <origin xyz="${scale_size*-0.25} ${scale_size*-0.11} ${scale_size*0.0}" rpy="0 0 0"/>
+        <origin xyz="${scale_size*-0.27} ${scale_size*-0.11} ${scale_size*0.0}" rpy="0 0 0"/>
         <axis xyz="1 0 0" />
     </joint>
@@ -178,5 +178,5 @@
         <parent link="base_link" />
         <child link="rear_left_thruster_link_nemesys" />
-        <origin xyz="${scale_size*-0.25} ${scale_size*0.11} ${scale_size*-0.0}" rpy="0 0 0"/>
+        <origin xyz="${scale_size*-0.27} ${scale_size*0.11} ${scale_size*-0.0}" rpy="0 0 0"/>
         <axis xyz="1 0 0" />
     </joint>
@@ -401,5 +401,5 @@
             <fluid_density>1000</fluid_density>
             <link name="base_link">
-                <center_of_volume>0 0 0</center_of_volume>
+                <center_of_volume>0 0 0.05</center_of_volume>
                 <volume>8.714e-3</volume>
             </link>
@@ -551,5 +551,5 @@
             <!-- Rotate so +X points to +Z (up) -->
             <pose>0 0 0 0 -1.570796 0</pose>
-            <visualize>true</visualize>
+            <visualize>false</visualize>
             <update_rate>10</update_rate>
             <ray>

Commit message: attacker control with cavepi

File: nemesys_surveillance/urdf/nemesys.urdf.xacro (robot description, xacro)
@@ -13,5 +13,5 @@
     <xacro:property name="negligible_volume" value="1.0e-9" />
     <material name="Custom_Color">
-        <color rgba="0.1 0.1 0.1 0.8" />
+        <color rgba="0.3 0.9 0.1 0.8" />
     </material>
     <material name="Orange">
@@ -382,5 +382,5 @@
     </gazebo>
     <gazebo reference="base_link">
-        <material>Gazebo/White</material>
+        <material>Gazebo/Green</material>
     </gazebo>
     <gazebo reference="front_right_thruster_link_nemesys">
@@ -443,5 +443,5 @@
         <plugin filename="libgazebo_ros_force.so" name="gazebo_ros_force">
             <bodyName>front_right_thruster_link_nemesys</bodyName>
-            <topicName>/front_right_thrust</topicName>
+            <topicName>/nemesys/front_right_thrust</topicName>
         </plugin>
     </gazebo>
@@ -449,5 +449,5 @@
         <plugin filename="libgazebo_ros_force.so" name="gazebo_ros_force">
             <bodyName>front_left_thruster_link_nemesys</bodyName>
-            <topicName>/front_left_thrust</topicName>
+            <topicName>/nemesys/front_left_thrust</topicName>
         </plugin>
     </gazebo>
@@ -455,5 +455,5 @@
         <plugin filename="libgazebo_ros_force.so" name="gazebo_ros_force">
             <bodyName>rear_right_thruster_link_nemesys</bodyName>
-            <topicName>/rear_right_thrust</topicName>
+            <topicName>/nemesys/rear_right_thrust</topicName>
         </plugin>
     </gazebo>
@@ -461,5 +461,5 @@
         <plugin filename="libgazebo_ros_force.so" name="gazebo_ros_force">
             <bodyName>rear_left_thruster_link_nemesys</bodyName>
-            <topicName>/rear_left_thrust</topicName>
+            <topicName>/nemesys/rear_left_thrust</topicName>
         </plugin>
     </gazebo>
@@ -467,5 +467,5 @@
         <plugin filename="libgazebo_ros_force.so" name="gazebo_ros_force">
             <bodyName>base_link</bodyName>
-            <topicName>/drag_force</topicName>
+            <topicName>/nemesys/drag_force</topicName>
         </plugin>
     </gazebo>
@@ -492,4 +492,5 @@
             </camera>
             <plugin name="camera_controller" filename="libgazebo_ros_camera.so">
+                <robotNamespace>/nemesys</robotNamespace>
                 <alwaysOn>true</alwaysOn>
                 <updateRate>0.0</updateRate>
@@ -530,4 +531,5 @@
             </camera>
             <plugin name="camera_controller" filename="libgazebo_ros_camera.so">
+                <robotNamespace>/nemesys</robotNamespace>
                 <alwaysOn>true</alwaysOn>
                 <updateRate>0.0</updateRate>
@@ -575,5 +577,5 @@
             </ray>
             <plugin name="gazebo_ros_laser" filename="libgazebo_ros_laser.so">
-            <topicName>/raw_depth_data</topicName>
+            <topicName>/nemesys/raw_depth_data</topicName>
             <frameName>bar30_sensor_link</frameName>
             </plugin>
@@ -589,5 +591,5 @@
             <topic>__default_topic__</topic>
             <plugin filename="libgazebo_ros_imu_sensor.so" name="imu_plugin">
-                <topicName>raw_imu_data</topicName>
+                <topicName>/nemesys/raw_imu_data</topicName>
                 <bodyName>imu_link</bodyName>
                 <updateRateHZ>10.0</updateRateHZ>
